Commit message: initial tuning

File: JakaCtrl/motion_policy_configs/Jaka/minicobo/minicobo_v14.urdf (robot description, URDF)
Before this commit: robot minicobo_v1.4, 9 links, 8 joints
Links:
- link Link0: mass 0.76174 -> 3.76174
- link Link4: mass 0.412340000009804 -> 1.412340000009804

File: JakaCtrl/motion_policy_configs/Jaka/minicobo/minicobo_v14_1.urdf (robot description, URDF)
Before this commit: robot minicobo_v1.4, 9 links, 8 joints
Links:
- link Link0: mass 0.76174 -> 3.76174
