Commit message: progress of a sort

File: JakaCtrl/motion_policy_configs/Jaka/minicobo/minicobo_v14_2.urdf (robot description, URDF)
Before this commit: robot minicobo_v1.4, 10 links, 9 joints
Joints:
- joint flange-tool0: parent dummy-tcp -> dummy_tcp

File: JakaCtrl/motion_policy_configs/Jaka/minicobo/minicobo_v14_onrobot_rg2.urdf (robot description, URDF)
Before this commit: robot minicobo_v1.4, 17 links, 16 joints
Links:
- removed link dummy_tcp
Joints:
- removed joint rs007n2rg2
- joint dummy_tcp_joint: child dummy_tcp -> onrobot_rg2_base_link
